File: CAN_H-Bridge_Solo_MD_fin.kicad_pcb (KiCad board)
At the start: 2 copper layers, 84.9 x 90.6 mm, 90 parts, among them IC1 SI8650AB-B-IS1, IC2 A3921KLPTR-T, J2 Conn_01x03, J3 Conn_01x05, J4 Bus_mechaken_PCIexpress_x16_1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, M1 Motor_DC, Q1 IRLB3813PBF, Q2 IRLB3813PBF, Q3 IRLB3813PBF, Q4 IRLB3813PBF, U1 LDL1117S33R_SOT223-4, U2 STM32F042K6Tx, U3 MCP2562-E-SN, U4 LDL1117S33TR_SOT223-4

Commit message: clean
Parts:
- added C14: 2.2u, Capacitor_SMD:C_0805_2012Metric_Pad1.15x1.40mm_HandSolder, B.Cu at (168.3, 84.8)
- added C14: 2.2u, Capacitor_SMD:C_0805_2012Metric_Pad1.15x1.40mm_HandSolder, B.Cu at (126.7, 138.7)
- added C15: 1u, Capacitor_SMD:C_0805_2012Metric_Pad1.15x1.40mm_HandSolder, B.Cu at (168.3, 79.2)
- added C15: 1u, Capacitor_SMD:C_0805_2012Metric_Pad1.15x1.40mm_HandSolder, B.Cu at (126.7, 144.3)
- added IC3: AP7381-50SA-7, SamacSys_Parts:SOT96P240X105-3N, B.Cu at (164.6, 82.8)
- added IC3: AP7381-50SA-7, SamacSys_Parts:SOT96P240X105-3N, B.Cu at (130.4, 140.8)
- C1 (x2), C10 (x2), C11 (x2), C12 (x2), C13 (x2), C2 (x2), C3 (x2), C4 (x2), C5 (x2), C6 (x2), C7 (x2), C8 (x2), C9 (x2): footprint Capacitor_SMD:C_0805_2012Metric -> Capacitor_SMD:C_0805_2012Metric_Pad1.15x1.40mm_HandSolder
- D1 (x2), D2 (x2), D3 (x2), D4 (x2): footprint LED_SMD:LED_0603_1608Metric -> LED_SMD:LED_0603_1608Metric_Castellated
- D5 (x2): footprint Diode_SMD:D_0603_1608Metric -> LED_SMD:LED_0603_1608Metric_Castellated
- J4 (x2): footprint PCIe:BUS_mechaken_PCIexpress_x16_164_Position -> PCIe:BUS_mechaken_PCIexpress_x16
- R1 (x2), R10 (x2), R11 (x2), R12 (x2), R2 (x2), R3 (x2), R4 (x2), R5 (x2), R6 (x2), R7 (x2), R8 (x2), R9 (x2): footprint Resistor_SMD:R_0603_1608Metric -> Resistor_SMD:R_0603_1608Metric_Pad1.05x0.95mm_HandSolder
- moved J4 91.0 mm to (189.0, 70.5), turned to 180 degrees
- moved D2 84.5 mm to (185.4, 107.7), turned to 180 degrees
- moved C1 83.8 mm to (187.7, 77.5), turned to 0 degrees
- moved C5 82.2 mm to (187.7, 80.7), turned to 180 degrees
- moved D1 81.9 mm to (185.4, 104.7), turned to 180 degrees
- moved R5 81.0 mm to (188.0, 89.5), turned to 90 degrees
- moved S1 77.4 mm to (183.0, 104.5), turned to 270 degrees
- moved R2 76.3 mm to (180.8, 107.7), turned to 180 degrees
- moved U1 73.9 mm to (183.8, 82.5), turned to 180 degrees
- moved R1 73.5 mm to (180.8, 104.7), turned to 180 degrees
- moved U2 72.5 mm to (183.0, 96.4), turned to 315 degrees
- moved C3 71.0 mm to (183.0, 88.5), turned to 180 degrees
- moved U3 69.6 mm to (181.1, 80.1), turned to 180 degrees
- moved R4 67.5 mm to (121.2, 111.0), turned to 180 degrees
- moved Q2 64.0 mm to (120.0, 106.5), turned to 180 degrees
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Routing:
- net VCC: track 65.2 -> 80.3 mm, vias 12 -> 16
- net GHB_0: track 43.9 -> 30.5 mm
- net GHA_0: track 35.4 -> 25.5 mm
- net MD_3V3: track 54.9 -> 64.2 mm, vias 0 -> 2
- net SA_0: track 47.7 -> 52.7 mm, vias 32 -> 30
- net SB_0: track 60.3 -> 55.6 mm, vias 34 -> 32
- net /SWCLK: track 60.8 -> 57.1 mm
- net Net-(Q3-Pad1): track 10.4 -> 13.9 mm
- net Net-(Q1-Pad1): track 10.3 -> 7.74 mm
- net VCP_RX: track 93.0 -> 90.8 mm
- net Net-(Q4-Pad1): track 10.2 -> 8.18 mm
- net Net-(Q2-Pad1): track 10.4 -> 8.49 mm
- net GLA_0: track 80.4 -> 78.9 mm
- net GNDPWR: track 89.4 -> 88.0 mm, vias 112 -> 122
- net GLB_0: track 87.2 -> 86.0 mm
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Other:
- board size 84.9 x 90.6 mm -> 84.3 x 72.6 mm
- board text added: "CAN H-Bridge Solo MD Prototype 1.1"
- board text added: "LED(ON:1 OFF:0) 00 -> Free 01 -> CW 10 -> CCW 11 -> Brake"
- board text added: "MSB"
- board text added: "Motor"
- board text removed: "CAN H-Bridge Solo MD Prototype 1.0"

Commit message: Release
Release Prototype-2.0
Parts:
- removed the C14 at (168.3, 84.8)
- removed the C14 at (126.7, 138.7)
- removed the C15 at (168.3, 79.2)
- removed the C15 at (126.7, 144.3)
- removed C4, C5: 0.1uF, Capacitor_SMD:C_0805_2012Metric_Pad1.15x1.40mm_HandSolder
- removed the D1 at (185.4, 104.7)
- removed IC1: SI8650AB-B-IS1, SamacSys_Parts:SOIC127P600X175-16N
- removed the IC3 at (164.6, 82.8)
- removed the IC3 at (130.4, 140.8)
- removed J4: Bus_mechaken_PCIexpress_x16_164_Position, PCIe:BUS_mechaken_PCIexpress_x16
- removed the Q1 at (141.1, 106.2)
- removed the Q1 at (153.9, 117.2)
- removed the Q2 at (120.0, 106.5)
- removed the Q2 at (175.0, 117.0)
- removed the Q3 at (141.0, 81.8)
- removed the Q3 at (154.0, 141.8)
- removed the Q4 at (120.0, 81.5)
- removed the Q4 at (175.0, 142.0)
- added C14: 0.1uF, Capacitor_SMD:C_0805_2012Metric_Pad1.15x1.40mm_HandSolder, F.Cu at (153.1, 92.0)
- added C15: 0.47uF, Capacitor_SMD:C_0805_2012Metric_Pad1.15x1.40mm_HandSolder, F.Cu at (157.9, 92.0)
- added D1: D_Schottky, Diode_SMD:D_0603_1608Metric_Pad1.05x0.95mm_HandSolder, F.Cu at (181.1, 73.3)
- added D1: D_Schottky, Diode_SMD:D_0603_1608Metric_Pad1.05x0.95mm_HandSolder, F.Cu at (103.9, 132.7)
- added D6: D, Diode_SMD:D_0603_1608Metric_Pad1.05x0.95mm_HandSolder, F.Cu at (147.6, 92.0)
- added IC3: A3921KLPTR-T, SamacSys_Parts:SOP65P640X120-29N, F.Cu at (152.0, 84.0)
- added J1: Conn_01x03, Connector_PinHeader_2.54mm:PinHeader_1x03_P2.54mm_Vertical, B.Cu at (149.9, 96.0)
- added Q1: TK6R7P06PLRQ, Package_TO_SOT_SMD:TO-252-2, B.Cu at (133.7, 95.0)
- added Q1: TK6R7P06PLRQ, Package_TO_SOT_SMD:TO-252-2, B.Cu at (151.3, 111.0)
- added Q2: TK6R7P06PLRQ, Package_TO_SOT_SMD:TO-252-2, B.Cu at (133.8, 70.9)
- added Q2: TK6R7P06PLRQ, Package_TO_SOT_SMD:TO-252-2, B.Cu at (151.2, 135.1)
- added Q3: TK6R7P06PLRQ, Package_TO_SOT_SMD:TO-252-2, B.Cu at (113.8, 95.1)
- added Q3: TK6R7P06PLRQ, Package_TO_SOT_SMD:TO-252-2, B.Cu at (171.2, 110.9)
- added Q4: TK6R7P06PLRQ, Package_TO_SOT_SMD:TO-252-2, B.Cu at (113.7, 70.8)
- added Q4: TK6R7P06PLRQ, Package_TO_SOT_SMD:TO-252-2, B.Cu at (171.3, 135.2)
- C1: value 1uF -> 0.1uF
- C10: value 0.47uF -> 4.7uF
- C11: value 1uF -> 4.7uF
- C12: value 0.1uF -> 4.7uF; moved to F.Cu
- C13, C8: value 4.7uF -> 0.1uF; moved to B.Cu
- C2, C6, C7: value 4.7uF -> 1uF
- C3: value 0.1uF -> 2.2uF
- C3: renamed from C2; value 4.7uF -> 2.2uF
- C7: renamed from C13; value 4.7uF -> 1uF
- C9: moved to B.Cu
- D5: value D -> LED
- D6: renamed from D5; footprint LED_SMD:LED_0603_1608Metric_Castellated -> Diode_SMD:D_0603_1608Metric_Pad1.05x0.95mm_HandSolder
- IC2: value A3921KLPTR-T -> SI8650AB-B-IS1; footprint SamacSys_Parts:SOP65P640X120-29N -> Package_SO:SOIC-16_3.9x9.9mm_P1.27mm
- IC2: renamed from IC1; footprint SamacSys_Parts:SOIC127P600X175-16N -> Package_SO:SOIC-16_3.9x9.9mm_P1.27mm
- J2: value Conn_01x03 -> Conthrough; footprint Connector_PinHeader_2.54mm:PinHeader_1x03_P2.54mm_Vertical -> Connector_PinHeader_2.54mm:PinHeader_1x05_P2.54mm_Vertical; moved to F.Cu
- J2: renamed from J3; value Conn_01x05 -> Conthrough
- J3: value Conn_01x05 -> Bus_mechaken_PCIexpress_x16_164_Position; footprint Connector_PinHeader_2.54mm:PinHeader_1x05_P2.54mm_Vertical -> PCIe:BUS_mechaken_PCIexpress_x16
- M1 (x2): moved to F.Cu
- R1: value 2.2K -> 10k
- R1: renamed from R5; value 10K -> 10k
- R10: value 3K -> 21; moved to F.Cu
- R11: value 10k -> 21; moved to F.Cu
- R12: value 2.2k -> 21; moved to F.Cu
- R2, R7: value 2.2K -> 2.2k
- R2: renamed from R1; value 2.2K -> 2.2k
- R3, R8: value 21 -> 2.2k
- R3: renamed from R2; value 2.2K -> 2.2k
- R4: value 21 -> 3k; moved to B.Cu
- R4: renamed from R10; value 3K -> 3k
- R5: value 10K -> 10k; moved to B.Cu
- R6: value 2.2K -> 2.2k; moved to B.Cu
- R7: renamed from R6; value 2.2K -> 2.2k
- R8: renamed from R7; value 2.2K -> 2.2k
- S1 (x2): value IKD0403101 -> DIPSW; footprint SamacSys_Parts:SOP254P980X370-8N -> Package_DIP:DIP-8_W7.62mm
- U1 (x2): value LDL1117S33R_SOT223-4 -> AP2210N-3.3TRG1; footprint Package_TO_SOT_SMD:SOT-223-3_TabPin2 -> Package_TO_SOT_SMD:SOT-23W_Handsoldering
- U2 (x2): value STM32F042K6Tx -> STM32F303K8
- U3: value MCP2562-E-SN -> MCP1799T-3302H/TT; footprint Package_SO:SOIC-8_3.9x4.9mm_P1.27mm -> Package_TO_SOT_SMD:SOT-23_Handsoldering; moved to F.Cu
- U3: renamed from U4; value LDL1117S33TR_SOT223-4 -> MCP1799T-3302H/TT; footprint Package_TO_SOT_SMD:SOT-223-3_TabPin2 -> Package_TO_SOT_SMD:SOT-23_Handsoldering
- U4: value LDL1117S33TR_SOT223-4 -> MCP2562-E-SN; footprint Package_TO_SOT_SMD:SOT-223-3_TabPin2 -> Package_SO:SOIC-8_3.9x4.9mm_P1.27mm; moved to B.Cu
- moved J3 54.0 mm to (184.0, 58.0), turned to 180 degrees
- moved R11 50.6 mm to (116.2, 100.8), turned to 180 degrees
- moved R4 49.2 mm to (161.0, 82.0), turned to 0 degrees
- moved C8 46.8 mm to (182.7, 68.2)
- moved D5 37.8 mm to (156.1, 66.8)
- moved C9 36.6 mm to (169.2, 69.6)
- moved R12 35.6 mm to (138.9, 140.0)
- moved C12 34.2 mm to (134.4, 85.0)
- moved R10 34.2 mm to (136.0, 78.2)
- moved R3 33.9 mm to (175.8, 97.8)
- moved C10 32.0 mm to (143.1, 79.4), turned to 180 degrees
- moved C6 30.7 mm to (162.8, 69.4)
- moved C11 30.5 mm to (143.1, 83.8), turned to 180 degrees
- moved R12 30.2 mm to (146.1, 66.0), turned to 0 degrees
- moved R5 28.9 mm to (161.0, 79.2), turned to 0 degrees
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- renumbered C3 to C1, C7 to C10, C6 to C11, C8 to C12, C12 to C13, C9 to C14, C10 to C15, C1 to C2, C11 to C6, C5 to C8, C4 to C9, D1 to D2, D2 to D3, D3 to D4, D4 to D5, IC2 to IC3, J2 to J1, J4 to J3, R8 to R10, R4 to R11, R9 to R12, R11 to R5, R12 to R6, R3 to R9, U3 to U4
Connections:
- C1 pad 1: +5V -> GND
- C1 pad 2: GND -> IC_3V3
- C1 pad 2: +3V3 -> IC_3V3
- C10 pad 2: Net-(C10-Pad2) -> SB_0
- C10 pad 1: Net-(C7-Pad1) -> Net-(C10-Pad1)
- C11 pad 1: VCC -> VREG_0
- C12 pad 1: V5 -> Net-(C12-Pad1)
- C12 pad 2: GNDPWR -> SA_0
- C12 pad 1: Net-(C8-Pad1) -> Net-(C12-Pad1)
- C13 pad 1: GNDPWR -> V5
- C13 pad 2: MD_3V3 -> GNDPWR
- C14 pad 1: Net-(C9-Pad1) -> Net-(C14-Pad1)
- C15 pad 1: Net-(C10-Pad1) -> Net-(C15-Pad1)
- C15 pad 2: Net-(C10-Pad2) -> Net-(C15-Pad2)
- C2 pad 1: GND -> +5V
- C2 pad 2: +3V3 -> GND
- C3 pad 2: +3V3 -> IC_3V3 (x2)
- C6 pad 1: VREG_0 -> VCC
- C7 pad 1: Net-(C7-Pad1) -> GNDPWR
- C7 pad 2: SB_0 -> MD_3V3
- C8 pad 1: Net-(C8-Pad1) -> GND
- C8 pad 2: SA_0 -> +5V
- C9 pad 1: Net-(C9-Pad1) -> GND
- C9 pad 2: GNDPWR -> IC_3V3
- C9 pad 2: +3V3 -> IC_3V3
- D2 pad 1: GND -> Net-(D2-Pad1) (x2)
- D2 pad 2: Net-(D2-Pad2) -> MD0_LED_H
- D2 pad 2: Net-(D1-Pad2) -> MD0_LED_H
- D3 pad 1: MD_FF1_0 -> Net-(D3-Pad1)
- D3 pad 2: Net-(D3-Pad2) -> MD0_LED_L
- D3 pad 1: GND -> Net-(D3-Pad1)
- D3 pad 2: Net-(D2-Pad2) -> MD0_LED_L
- D4 pad 1: MD_FF2_0 -> MD_FF1_0
- D4 pad 2: Net-(D3-Pad2) -> Net-(D4-Pad2)
- D5 pad 1: Net-(C9-Pad1) -> MD_FF2_0
- D5 pad 2: VCC -> Net-(D5-Pad2)
- D5 pad 2: Net-(D4-Pad2) -> Net-(D5-Pad2)
- D6 pad 1: Net-(C9-Pad1) -> Net-(C14-Pad1)
- IC2 pad 1: VCC -> IC_3V3
- IC2 pad 10: GHA_0 -> MD_3V3
- IC2 pad 11: SA_0 -> MD_RESET_0
- IC2 pad 12: GLA_0 -> MD_PWMH_0
- IC2 pad 13: Net-(C9-Pad1) -> MD_PWML_0
- IC2 pad 14: Net-(IC2-Pad14) -> MD_SR_0
- IC2 pad 15: Net-(C10-Pad1) -> MD_PHASE_0
- IC2 pad 16: Net-(C10-Pad2) -> MD_3V3
- IC2 pad 2: GNDPWR -> IC_PHASE_0
- IC2 pad 3: GLB_0 -> IC_SR_0
- IC2 pad 4: SB_0 -> IC_PWML_0
- IC2 pad 5: GHB_0 -> IC_PWMH_0
- IC2 pad 6: Net-(C7-Pad1) -> IC_RESET_0
- IC2 pad 8: VREG_0 -> GND
- IC2 pad 9: Net-(C8-Pad1) -> GNDPWR
- IC2 pad 1: +3V3 -> IC_3V3
- IC2 pad 10: Net-(IC1-Pad10) -> MD_3V3
- IC2 pad 7: Net-(IC1-Pad7) -> Net-(IC2-Pad7)
- IC3 pad 13: Net-(C9-Pad1) -> Net-(C14-Pad1)
- IC3 pad 14: Net-(IC2-Pad14) -> Net-(IC3-Pad14)
- IC3 pad 15: Net-(C10-Pad1) -> Net-(C15-Pad1)
- IC3 pad 16: Net-(C10-Pad2) -> Net-(C15-Pad2)
- IC3 pad 18: Net-(IC2-Pad18) -> Net-(IC3-Pad18)
- IC3 pad 27: Net-(IC2-Pad27) -> Net-(IC3-Pad27)
- IC3 pad 28: Net-(IC2-Pad28) -> Net-(IC3-Pad28)
- IC3 pad 6: Net-(C7-Pad1) -> Net-(C10-Pad1)
- IC3 pad 7: Net-(IC2-Pad7) -> Net-(IC3-Pad7)
- IC3 pad 9: Net-(C8-Pad1) -> Net-(C12-Pad1)
- J2 pad 1: GND -> NRST
- J2 pad 2: VCP_TX -> /SWDIO
- J2 pad 3: VCP_RX -> GND
- J2 pad 5: +3V3 -> IC_3V3
- J3 pad A5: Net-(J4-PadA5) -> Net-(J3-PadA5)
- J3 pad A6: Net-(J4-PadA6) -> Net-(J3-PadA6)
- J3 pad A7: Net-(J4-PadA7) -> Net-(J3-PadA7)
- J3 pad B3: Net-(J4-PadB3) -> Net-(J3-PadB3)
- J3 pad B4: Net-(J4-PadB4) -> Net-(J3-PadB4)
- J3 pad B5: Net-(J4-PadB5) -> Net-(J3-PadB5)
- J3 pad B6: Net-(J4-PadB6) -> Net-(J3-PadB6)
- J3 pad B7: Net-(J4-PadB7) -> Net-(J3-PadB7)
- J3 pad B9: Net-(J4-PadB9) -> VCC
- M1 pad 1: SB_0 -> SA_0 (x2)
- M1 pad 2: SA_0 -> SB_0 (x2)
- R1 pad 1: Net-(D1-Pad2) -> /BOOT
- R1 pad 2: MD0_LED_H -> GND
- R10 pad 1: Net-(IC2-Pad27) -> Net-(Q2-Pad1)
- R10 pad 2: V5 -> GHB_0
- R10 pad 1: Net-(Q3-Pad1) -> Net-(Q2-Pad1)
- R11 pad 1: Net-(IC2-Pad28) -> GLA_0
- R11 pad 2: V5 -> Net-(Q3-Pad1)
- R11 pad 2: Net-(Q2-Pad1) -> Net-(Q3-Pad1)
- R12 pad 1: GNDPWR -> Net-(Q4-Pad1)
- R12 pad 2: Net-(IC2-Pad28) -> GLB_0
- R2 pad 1: Net-(D2-Pad2) -> Net-(D2-Pad1)
- R2 pad 2: MD0_LED_L -> GND
- R2 pad 1: Net-(D1-Pad2) -> Net-(D2-Pad1)
- R2 pad 2: MD0_LED_H -> GND
- R3 pad 1: GHA_0 -> Net-(D3-Pad1)
- R3 pad 2: Net-(Q1-Pad1) -> GND
- R3 pad 1: Net-(D2-Pad2) -> Net-(D3-Pad1)
- R3 pad 2: MD0_LED_L -> GND
- R4 pad 1: GLA_0 -> Net-(IC3-Pad27)
- R4 pad 2: Net-(Q2-Pad1) -> V5
- R4 pad 1: Net-(IC2-Pad27) -> Net-(IC3-Pad27)
- R5 pad 1: /BOOT -> Net-(IC3-Pad28)
- R5 pad 2: GND -> V5
- R5 pad 1: Net-(IC2-Pad28) -> Net-(IC3-Pad28)
- R6 pad 1: V5 -> GNDPWR
- R6 pad 2: Net-(D3-Pad2) -> Net-(IC3-Pad28)
- R6 pad 2: Net-(IC2-Pad28) -> Net-(IC3-Pad28)
- R7 pad 2: Net-(D3-Pad2) -> Net-(D4-Pad2)
- R8 pad 1: Net-(Q3-Pad1) -> V5
- R8 pad 2: GHB_0 -> Net-(D5-Pad2)
- R8 pad 2: Net-(D4-Pad2) -> Net-(D5-Pad2)
- R9 pad 1: Net-(Q4-Pad1) -> GHA_0
- R9 pad 2: GLB_0 -> Net-(Q1-Pad1)
- S1 pad 5: +3V3 -> IC_3V3 (x2)
- S1 pad 6: +3V3 -> IC_3V3 (x2)
- S1 pad 7: +3V3 -> IC_3V3 (x2)
- S1 pad 8: +3V3 -> IC_3V3 (x2)
- U1 pad 2: +3V3 -> IC_3V3 (x2)
- U2 pad 1: +3V3 -> IC_3V3 (x2)
- U2 pad 17: +3V3 -> IC_3V3 (x2)
- U2 pad 19: MD0_LED_L -> MD0_LED_H (x2)
- U2 pad 20: MD0_LED_H -> MD0_LED_L (x2)
- U2 pad 5: +3V3 -> IC_3V3 (x2)
- U3 pad 1: /CAN_TD -> GNDPWR
- U3 pad 2: GND -> MD_3V3
- U3 pad 3: +5V -> VCC
- U4 pad 1: GNDPWR -> /CAN_TD
- U4 pad 2: MD_3V3 -> GND
- U4 pad 3: VCC -> +5V
- U4 pad 5: +3V3 -> IC_3V3
Routing:
- net IC_3V3: track 0.00 -> 160.5 mm, vias 0 -> 6
- net +3V3: track 139.5 -> 0.00 mm, vias 6 -> 0
- net Net-(Q4-Pad1): track 8.18 -> 82.4 mm, vias 0 -> 2
- net Net-(J4-PadB9): track 58.2 -> 0.00 mm
- net GLB_0: track 86.0 -> 33.0 mm
- net SB_0: track 55.6 -> 93.3 mm, vias 32 -> 224
- net GNDPWR: track 88.0 -> 122.5 mm, vias 122 -> 190
- net VCC: track 80.3 -> 111.4 mm, vias 16 -> 396
- net Net-(Q1-Pad1): track 7.74 -> 35.4 mm, vias 0 -> 2
- net Net-(C12-Pad1): track 0.00 -> 27.3 mm
- net MD_3V3: track 64.2 -> 39.0 mm, vias 2 -> 0
- net MD_FF2_0: track 13.3 -> 33.2 mm
- net Net-(C14-Pad1): track 0.00 -> 19.7 mm
- net Net-(C9-Pad1): track 18.6 -> 0.00 mm
- net /SWCLK: track 57.1 -> 75.1 mm
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- added copper zone on F.Cu, net VCC
Other:
- board size 84.3 x 72.6 mm -> 84.3 x 80.1 mm
- board text added: "CAN H-Bridge Solo MD Prototype 2.0"
- board text added: "FF1"
- board text added: "FF2"
- board text added: "https://github.com/picopicodevil/CAN_H-Bridge_Solo_MD.git"
- board text removed: "CAN H-Bridge Solo MD Prototype 1.1"
